File: PCB/Ducky.kicad_sch (KiCad schematic)
At the start: 10 parts, among them J1 Conn_01x22_Socket, J2 Conn_01x22_Socket, SW1 On/Off Button, SW2 Recording/Stop Recording Butt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, U1 ESP32-S3-DEVKITC-1-N8R2

Commit message: I am organzing my folders and files
Parts:
- added J3: Conn_01x06_Socket, Connector_PinSocket_2.54mm:PinSocket_1x06_P2.54mm_Vertical, symbol Connector:Conn_01x06_Socket
- renumbered GLED to GLED1, RLED to RLED1
Connections:
- net +3V3: now also J3.1 (Pin_1); no longer U1.J1_1 (3V3), U1.J1_2 (3V3)
- net GND: now also J3.6 (Pin_6)
- net CS: now reaches J1.16 (Pin_16)
- net CS: now also J3.2 (Pin_2)
- net MOSI: now reaches J1.17 (Pin_17)
- net MOSI: now also J3.3 (Pin_3)
- net CLK: now reaches J1.18 (Pin_18)
- net CLK: now also J3.4 (Pin_4)
- net MISO: now reaches J1.19 (Pin_19)
- net MISO: now also J3.5 (Pin_5)
- new net 3V3: U1.J1_1 (3V3), U1.J1_2 (3V3)
- no-connect marks 52 -> 49
